File: foam/eugeo-case-foam.kicad_pcb (KiCad board)
At the start: 2 copper layers, 114.4 x 76.4 mm, 0 parts

Commit message: Add Yushakobo laser-cut SVGs and pre-order checks
- lasercut/yushakobo: centre cover (clear acrylic 2 mm), switch plates
  (POM 1.5 mm) and plate/case foams (PORON 3 mm) laid out on Yushakobo's
  official Inkscape templates, with export and rule-check scripts
- plate foam: 3 mm PORON, standoff holes 4.4 mm to keep a 1 mm web
- scripts/preorder_check.py: revision diff, placement, hardware vs exposed
  copper, via tenting, JLCPCB minimums, Gerber freshness, drill/CPL/plate
  alignment, laser-cut SVG rules and functional checks (22/22 pass)

Co-Authored-By: Claude Opus 5.5 <noreply@anthropic.com>
Other:
- board text added: "eugeo case foam - cut 2 (flip one), 3 mm PORON"
- board text removed: "eugeo case foam - cut 2 (flip one), 3 mm PORON / EVA"
Changed lines of the file:
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@@
-	)
-	(gr_line
-		(start 129.4 161.094)
-		(end 129.4 165.094)
-		(stroke
-			(width 0.2)
-			(type default)
-		)
-		(layer "Dwgs.User")
 	)
 	(gr_line
@@
 		(layer "Dwgs.User")
 	)
-	(gr_arc
-		(start 142.3 74.694)
-		(mid 143.36066 75.13334)
-		(end 143.8 76.194)
+	(gr_line
+		(start 129.4 161.094)
+		(end 129.4 165.094)
 		(stroke
-			(width 0.1)
+			(width 0.2)
 			(type default)
 		)
-		(layer "Edge.Cuts")
+		(layer "Dwgs.User")
 	)
 	(gr_arc
@@
 	)
 	(gr_line
-		(start 29.45 149.544)
-		(end 29.45 76.194)
-		(stroke
-			(width 0.1)
-			(type default)
-		)
-		(layer "Edge.Cuts")
-	)
-	(gr_line
-		(start 30.95 74.694)
-		(end 142.3 74.694)
-		(stroke
-			(width 0.1)
-			(type default)
-		)
-		(layer "Edge.Cuts")
-	)
-	(gr_arc
-		(start 30.95 151.044)
-		(mid 29.88934 150.60466)
-		(end 29.45 149.544)
-		(stroke
-			(width 0.1)
-			(type default)
-		)
-		(layer "Edge.Cuts")
-	)
-	(gr_line
 		(start 143.8 76.194)
 		(end 143.8 149.544)
-		(stroke
-			(width 0.1)
-			(type default)
-		)
-		(layer "Edge.Cuts")
-	)
-	(gr_arc
-		(start 143.8 149.544)
-		(mid 143.36066 150.60466)
-		(end 142.3 151.044)
 		(stroke
 			(width 0.1)
@@
 		(layer "Edge.Cuts")
 	)
+	(gr_line
+		(start 30.95 74.694)
+		(end 142.3 74.694)
+		(stroke
+			(width 0.1)
+			(type default)
+		)
+		(layer "Edge.Cuts")
+	)
 	(gr_circle
 		(center 124.775 93.819)
@@
 		)
 		(fill no)
+		(layer "Edge.Cuts")
+	)
+	(gr_line
+		(start 29.45 149.544)
+		(end 29.45 76.194)
+		(stroke
+			(width 0.1)
+			(type default)
+		)
+		(layer "Edge.Cuts")
+	)
+	(gr_arc
+		(start 143.8 149.544)
+		(mid 143.36066 150.60466)
+		(end 142.3 151.044)
+		(stroke
+			(width 0.1)
+			(type default)
+		)
 		(layer "Edge.Cuts")
 	)
@@
 		(layer "Edge.Cuts")
 	)
+	(gr_arc
+		(start 142.3 74.694)
+		(mid 143.36066 75.13334)
+		(end 143.8 76.194)
+		(stroke
+			(width 0.1)
+			(type default)
+		)
+		(layer "Edge.Cuts")
+	)
+	(gr_arc
+		(start 30.95 151.044)
+		(mid 29.88934 150.60466)
+		(end 29.45 149.544)
+		(stroke
+			(width 0.1)
+			(type default)
+		)
+		(layer "Edge.Cuts")
+	)
 	(gr_text "100 mm (print at 100% / actual size)"
 		(at 29.4 168.094 0)
@@
 		)
 	)
-	(gr_text "eugeo case foam - cut 2 (flip one), 3 mm PORON / EVA"
+	(gr_text "eugeo case foam - cut 2 (flip one), 3 mm PORON"
 		(at 29.4 173.094 0)
 		(layer "Dwgs.User")
