File: eugeo.kicad_pcb (KiCad board)
At the start: 2 copper layers, 284.9 x 75.4 mm, 143 parts, among them J1 USB-C, SW1 RESET, SW2 BOOT, U1 RP2040, U2 W25Q16JVSSIQ, U3 MCP1700-3302E, U4 USBLC6-2SC6, Y1 12MHz

Commit message: Cover screws at the corners and a large EUGEO logo on the back
- Centre cover holes move to the four corners of the acrylic
  (131.5 / 173.3 x 59.4 / 126.3). The column buses along the bottom edge
  split around the lower screws: COL5 / COL4 above, COL3..COL0 below.
- Back side: Futura "EUGEO" (same face as the case nameplate), 7.5 mm cap
  height with a rule and dot each side, in the free band between key rows
  1 and 2. Letters are pre-outlined by scripts/logo_outline.py into
  scripts/logo_eugeo.json and drawn by stump_art.py, which keeps the frost
  and snowflakes clear of it.
- Cover, plates, laser-cut SVGs, case and renders regenerated.

Co-Authored-By: Claude Opus 5.5 <noreply@anthropic.com>
Parts:
- moved H12 13.4 mm to (173.3, 126.3)
- moved H11 13.4 mm to (131.5, 126.3)
Routing:
- net /CONN_D+: track 30.8 -> 21.3 mm, vias 1 -> 2
- net /COL3: track 334.3 -> 340.3 mm
- net /VBUS: track 46.3 -> 40.4 mm
- net +5V: track 57.8 -> 63.2 mm, vias 1 -> 0
- net /COL2: track 373.6 -> 378.4 mm
- net /COL1: track 415.6 -> 419.2 mm
- net /QSPI_SS: track 46.7 -> 43.7 mm
- net /COL0: track 457.6 -> 460.0 mm
- net /COL4: track 292.3 -> 290.7 mm
- net +3V3: track 76.6 -> 77.3 mm
